Commit message: wip: debugging initial state, and reset state

File: assets/urdf/vss_robot.urdf (robot description, URDF)
Before this commit: robot vss_robot, 3 links, 2 joints
Links:
- removed link left_wheel
- removed link right_wheel
- link robot_body: mass 1 -> None; geometry collision box size=0.1 0.1 0.1; visual box size=0.1 0.1 0.1
Joints:
- removed joint left_wheel_axis
- removed joint right_wheel_axis
