Commit message: vss robot with differential drive

File: assets/rsoccer/vss_robot.urdf (robot description, URDF)
Before this commit: robot vss_robot, 1 links, 0 joints
Links:
- added link left_wheel
- added link right_wheel
- link robot_body: mass None -> 0.150; geometry collision box size=0.08 0.075 0.055; visual box size=0.08 0.075 0.055
Joints:
- added joint left_wheel_joint: type fixed, parent robot_body, child left_wheel, origin xyz=0.0 0.04 -0.004
- added joint right_wheel_joint: type fixed, parent robot_body, child right_wheel, origin xyz=0.0 -0.04 -0.004

Commit message: vss wheel visual and test script

File: assets/rsoccer/vss_robot.urdf (robot description, URDF)
Before this commit: robot vss_robot, 3 links, 2 joints
Links:
- link left_wheel: geometry visual cylinder length=0.0025 radius=0.026
- link right_wheel: geometry visual cylinder length=0.0025 radius=0.026
