Commit message: add ball grad and make ball collidable

File: assets/rsoccer/golf_ball.urdf (robot description, URDF)
Before this commit: robot ball, 1 links, 0 joints
Links:
- link ball: geometry collision sphere radius=0.02134; visual sphere radius=0.02134

Commit message: add wheeled robot to v1

File: assets/rsoccer/golf_ball.urdf (robot description, URDF)
Before this commit: robot ball, 1 links, 0 joints
Links:
- link ball: mass None -> 0.04593
