Commit message: change robot properties so it does not move when tumbled

File: isaacgymenvs/tasks/rsoccer/assets/vss_robot.urdf (robot description, URDF)
Before this commit: robot vss, 5 links, 4 joints
Links:
- link body: mass 0.330 -> 0.4; geometry collision box size=0.07 0.07 0.056; visual box size=0.07 0.06 0.056
Joints:
- joint body_leftWheel: origin xyz=0.0 0.03375 0.002 rpy=-1.570796 0.0 0.0 -> xyz=0.0 0.03375 -0.005 rpy=-1.570796 0.0 0.0
- joint body_rightWheel: origin xyz=0.0 -0.03375 0.002 rpy=-1.570796 0.0 0.0 -> xyz=0.0 -0.03375 -0.005 rpy=-1.570796 0.0 0.0
- joint body_tagId: origin xyz=0.0175 0.0 0.021 -> xyz=0.0175 0.0 0.028
- joint body_tagTeam: origin xyz=-0.0175 0.0 0.021 -> xyz=-0.0175 0.0 0.028

Commit message: revert robot physics change

File: isaacgymenvs/tasks/rsoccer/assets/vss_robot.urdf (robot description, URDF)
Before this commit: robot vss, 5 links, 4 joints
Links:
- link body: mass 0.4 -> 0.330; geometry collision box size=0.07 0.07 0.042; visual box size=0.07 0.06 0.042
Joints:
- joint body_leftWheel: origin xyz=0.0 0.03375 -0.005 rpy=-1.570796 0.0 0.0 -> xyz=0.0 0.03375 0.002 rpy=-1.570796 0.0 0.0
- joint body_rightWheel: origin xyz=0.0 -0.03375 -0.005 rpy=-1.570796 0.0 0.0 -> xyz=0.0 -0.03375 0.002 rpy=-1.570796 0.0 0.0
- joint body_tagId: origin xyz=0.0175 0.0 0.028 -> xyz=0.0175 0.0 0.021
- joint body_tagTeam: origin xyz=-0.0175 0.0 0.028 -> xyz=-0.0175 0.0 0.021
